Commit message: add keypoint1 in gripper_single_urdf.xacro

File: pr2_description/urdf/gripper_v0/gripper_single.urdf.xacro (robot description, xacro)
@@ -12,4 +12,7 @@
   <xacro:property name="finger_to_finger_tip_x"     value="0.09137" />
   <xacro:property name="palm_to_finger_x"           value="0.07691" />
+  <xacro:property name="keypoint1_both_x" value="0.071" />
+  <xacro:property name="keypoint1_l_y" value="0.0032" />
+  <xacro:property name="keypoint1_r_y" value="-{keypoint1_l_y}" />
   <xacro:macro name="pr2_finger_limits_v0">
     <!-- limits on passive finger and finger top joints without
@@ -56,4 +59,14 @@
       </collision>
     </link>
+    <joint name="${prefix}_l_keypoint1_joint" type="revolute">
+      <axis xyz="0 0 1" />
+      <!-- <origin xyz="${0.09137} ${-0.00495} 0" rpy="0 0 0" /> -->
+      <origin xyz="${keypoint1_both_x} ${keypoint1_l_y} 0.0" rpy="0 0 0" />
+      <xacro:pr2_finger_limits_v0/>
+      <dynamics damping="${finger_tip_damping}" />
+      <parent link="${prefix}_l_finger_link"/>
+      <child link="${prefix}_l_keypoint1_link"/>
+    </joint>
+    <link name="${prefix}_l_keypoint1_link"/>
     <!-- Finger proximal digit -->
     <joint name="${prefix}_r_finger_joint" type="revolute">
@@ -155,14 +168,18 @@
       </collision>
     </link>
+    <joint name="${prefix}_r_keypoint1_joint" type="revolute">
+      <axis xyz="0 0 1" />
+      <!-- <origin xyz="${0.09137} ${-0.00495} 0" rpy="0 0 0" /> -->
+      <origin xyz="${0.071} ${-0.0032} 0.0" rpy="0 0 0" />
+      <xacro:pr2_finger_limits_v0/>
+      <dynamics damping="${finger_tip_damping}" />
+      <parent link="${prefix}_r_finger_link"/>
+      <child link="${prefix}_r_keypoint1_link"/>
+    </joint>
+    <link name="${prefix}_r_keypoint1_link"/>
     <!-- extensions -->
     <xacro:pr2_finger_gazebo_v0 prefix="${prefix}" reflect="${reflect}" />
   </xacro:macro>
   <xacro:macro name="pr2_gripper_v0" params="side reflect name *origin gear_ratio screw_reduction theta0 phi0 t0 L0 h a b r">
-    <!-- <joint name="${side}_gripper_palm_joint" type="fixed"> -->
-    <!--   <xacro:insert_block name="origin"/> -->
-    <!--   <parent link="${parent}"/> -->
-    <!--   <child link="${side}_gripper_palm_link"/> -->
-    <!-- </joint> -->
-    <!-- <link name="${side}_gripper_palm_link"> -->
     <link name="${name}_link">
       <inertial>

Commit message: add keypoint2

File: pr2_description/urdf/gripper_v0/gripper_single.urdf.xacro (robot description, xacro)
@@ -14,5 +14,8 @@
   <xacro:property name="keypoint1_both_x" value="0.071" />
   <xacro:property name="keypoint1_l_y" value="0.0032" />
-  <xacro:property name="keypoint1_r_y" value="-{keypoint1_l_y}" />
+  <xacro:property name="keypoint1_r_y" value="-${keypoint1_l_y}" />
+  <xacro:property name="keypoint2_both_x" value="0.119" />
+  <xacro:property name="keypoint2_l_y" value="0.007" />
+  <xacro:property name="keypoint2_r_y" value="-${keypoint2_l_y}" />
   <xacro:macro name="pr2_finger_limits_v0">
     <!-- limits on passive finger and finger top joints without
@@ -165,5 +168,5 @@
         <geometry>
           <mesh filename="package://pr2_description/meshes/gripper_v0/l_finger_tip.stl"  />
-        </geometry>
+NN        </geometry>
       </collision>
     </link>
@@ -243,4 +246,18 @@
     </joint>
     <link name="${side}_gripper_tool_frame"/>
+    <joint name="${side}_gripper_l_keypoint2_joint" type="fixed">
+      <axis xyz="0 0 1" />
+      <origin xyz="${keypoint2_both_x} ${keypoint2_l_y} 0.0" rpy="0 0 0" />
+      <parent link="${name}_link"/>
+      <child link="${side}_gripper_l_keypoint2_link"/>
+    </joint>
+    <link name="${side}_gripper_l_keypoint2_link"/>
+    <joint name="${side}_gripper_r_keypoint2_joint" type="fixed">
+      <axis xyz="0 0 1" />
+      <origin xyz="${keypoint2_both_x} ${keypoint2_r_y} 0.0" rpy="0 0 0" />
+      <parent link="${name}_link"/>
+      <child link="${side}_gripper_r_keypoint2_link"/>
+    </joint>
+    <link name="${side}_gripper_r_keypoint2_link"/>
     <!-- actuated motor screw joint -->
     <link name="${side}_gripper_motor_slider_link">

Commit message: add keypoint3

File: pr2_description/urdf/gripper_v0/gripper_single.urdf.xacro (robot description, xacro)
@@ -18,4 +18,7 @@
   <xacro:property name="keypoint2_l_y" value="0.007" />
   <xacro:property name="keypoint2_r_y" value="-${keypoint2_l_y}" />
+  <xacro:property name="keypoint3_both_x" value="0.024" />
+  <xacro:property name="keypoint3_l_y" value="-${keypoint3_r_y}" />
+  <xacro:property name="keypoint3_r_y" value="0.006" />
   <xacro:macro name="pr2_finger_limits_v0">
     <!-- limits on passive finger and finger top joints without
@@ -139,4 +142,26 @@
       </collision>
     </link>
+    <joint name="${side}_gripper_l_joint" type="prismatic">
+      <parent link="${side}_gripper_l_finger_tip_link"/>
+      <child link="${side}_gripper_l_finger_tip_frame"/>
+      <axis xyz="0 1 0" />
+      <dynamics damping="${gripper_damping}" />
+      <limit effort="1000.0" velocity="0.2" lower="0.0" upper="0.09" />
+      <safety_controller k_velocity="5000.0" k_position="20.0" soft_lower_limit="${0.0-0.01}" soft_upper_limit="${0.09-0.002}" />
+    </joint>
+    <!-- This link is the same as the l_finger_tip_link,
+	 but because the urdf does not support graph structures,
+	 this link exists twice -->
+    <link name="${side}_gripper_l_finger_tip_frame" />
+    <joint name="${side}_gripper_l_keypoint3_joint" type="fixed">
+      <axis xyz="0 0 1" />
+      <!-- <origin xyz="${0.09137} ${-0.00495} 0" rpy="0 0 0" /> -->
+      <origin xyz="${keypoint3_both_x} ${keypoint3_l_y} 0.0" rpy="0 0 0" />
+      <xacro:pr2_finger_limits_v0/>
+      <dynamics damping="${finger_tip_damping}" />
+      <parent link="${side}_gripper_l_finger_tip_frame"/>
+      <child link="${side}_gripper_l_keypoint3_link"/>
+    </joint>
+    <link name="${side}_gripper_l_keypoint3_link"/>
     <!-- Finger tip -->
     <joint name="${prefix}_r_finger_tip_joint" type="revolute">
@@ -168,5 +193,5 @@
         <geometry>
           <mesh filename="package://pr2_description/meshes/gripper_v0/l_finger_tip.stl"  />
-NN        </geometry>
+        </geometry>
       </collision>
     </link>
@@ -331,7 +356,7 @@
          k_velocity was recently raised from 500.0 to 5000.0.  Tested on beta
     -->
-    <joint name="${side}_gripper_joint" type="prismatic">
+    <joint name="${side}_gripper_r_joint" type="prismatic">
       <parent link="${side}_gripper_r_finger_tip_link"/>
-      <child link="${side}_gripper_l_finger_tip_frame"/>
+      <child link="${side}_gripper_r_finger_tip_frame"/>
       <axis xyz="0 1 0" />
       <dynamics damping="${gripper_damping}" />
@@ -342,5 +367,15 @@
 	 but because the urdf does not support graph structures,
 	 this link exists twice -->
-    <link name="${side}_gripper_l_finger_tip_frame" />
+    <link name="${side}_gripper_r_finger_tip_frame" />
+    <joint name="${side}_gripper_r_keypoint3_joint" type="fixed">
+      <axis xyz="0 0 1" />
+      <!-- <origin xyz="${0.09137} ${-0.00495} 0" rpy="0 0 0" /> -->
+      <origin xyz="${keypoint3_both_x} ${keypoint3_r_y} 0.0" rpy="0 0 0" />
+      <xacro:pr2_finger_limits_v0/>
+      <dynamics damping="${finger_tip_damping}" />
+      <parent link="${side}_gripper_r_finger_tip_frame"/>
+      <child link="${side}_gripper_r_keypoint3_link"/>
+    </joint>
+    <link name="${side}_gripper_r_keypoint3_link"/>
     <!-- extensions -->
     <xacro:pr2_gripper_gazebo_v0 side="${side}" />

Commit message: add keypoint4

File: pr2_description/urdf/gripper_v0/gripper_single.urdf.xacro (robot description, xacro)
@@ -21,4 +21,7 @@
   <xacro:property name="keypoint3_l_y" value="-${keypoint3_r_y}" />
   <xacro:property name="keypoint3_r_y" value="0.006" />
+  <xacro:property name="keypoint4_both_x" value="0.0115" />
+  <xacro:property name="keypoint4_l_y" value="0.0032" />
+  <xacro:property name="keypoint4_r_y" value="-${keypoint4_l_y}" />
   <xacro:macro name="pr2_finger_limits_v0">
     <!-- limits on passive finger and finger top joints without
@@ -164,4 +167,14 @@
     </joint>
     <link name="${side}_gripper_l_keypoint3_link"/>
+    <joint name="${side}_gripper_l_keypoint4_joint" type="fixed">
+      <axis xyz="0 0 1" />
+      <!-- <origin xyz="${0.09137} ${-0.00495} 0" rpy="0 0 0" /> -->
+      <origin xyz="${keypoint4_both_x} ${keypoint4_l_y} 0.0" rpy="0 0 0" />
+      <xacro:pr2_finger_limits_v0/>
+      <dynamics damping="${finger_tip_damping}" />
+      <parent link="${side}_gripper_l_finger_tip_frame"/>
+      <child link="${side}_gripper_l_keypoint4_link"/>
+    </joint>
+    <link name="${side}_gripper_l_keypoint4_link"/>
     <!-- Finger tip -->
     <joint name="${prefix}_r_finger_tip_joint" type="revolute">
@@ -378,4 +391,14 @@
     </joint>
     <link name="${side}_gripper_r_keypoint3_link"/>
+    <joint name="${side}_gripper_r_keypoint4_joint" type="fixed">
+      <axis xyz="0 0 1" />
+      <!-- <origin xyz="${0.09137} ${-0.00495} 0" rpy="0 0 0" /> -->
+      <origin xyz="${keypoint4_both_x} ${keypoint4_r_y} 0.0" rpy="0 0 0" />
+      <xacro:pr2_finger_limits_v0/>
+      <dynamics damping="${finger_tip_damping}" />
+      <parent link="${side}_gripper_r_finger_tip_frame"/>
+      <child link="${side}_gripper_r_keypoint4_link"/>
+    </joint>
+    <link name="${side}_gripper_r_keypoint4_link"/>
     <!-- extensions -->
     <xacro:pr2_gripper_gazebo_v0 side="${side}" />

Commit message: change keypoint1 fixed

File: pr2_description/urdf/gripper_v0/gripper_single.urdf.xacro (robot description, xacro)
@@ -68,5 +68,5 @@
       </collision>
     </link>
-    <joint name="${prefix}_l_keypoint1_joint" type="revolute">
+    <joint name="${prefix}_l_keypoint1_joint" type="fixed">
       <axis xyz="0 0 1" />
       <!-- <origin xyz="${0.09137} ${-0.00495} 0" rpy="0 0 0" /> -->
@@ -209,5 +209,5 @@
       </collision>
     </link>
-    <joint name="${prefix}_r_keypoint1_joint" type="revolute">
+    <joint name="${prefix}_r_keypoint1_joint" type="fixed">
       <axis xyz="0 0 1" />
       <!-- <origin xyz="${0.09137} ${-0.00495} 0" rpy="0 0 0" /> -->

Commit message: change parent of kp3&4

File: pr2_description/urdf/gripper_v0/gripper_single.urdf.xacro (robot description, xacro)
@@ -145,4 +145,24 @@
       </collision>
     </link>
+    <joint name="${side}_gripper_l_keypoint3_joint" type="fixed">
+      <axis xyz="0 0 1" />
+      <!-- <origin xyz="${0.09137} ${-0.00495} 0" rpy="0 0 0" /> -->
+      <origin xyz="${keypoint3_both_x} ${keypoint3_l_y} 0.0" rpy="0 0 0" />
+      <xacro:pr2_finger_limits_v0/>
+      <dynamics damping="${finger_tip_damping}" />
+      <parent link="${side}_gripper_l_finger_tip_link"/>
+      <child link="${side}_gripper_l_keypoint3_link"/>
+    </joint>
+    <link name="${side}_gripper_l_keypoint3_link"/>
+    <joint name="${side}_gripper_l_keypoint4_joint" type="fixed">
+      <axis xyz="0 0 1" />
+      <!-- <origin xyz="${0.09137} ${-0.00495} 0" rpy="0 0 0" /> -->
+      <origin xyz="${keypoint4_both_x} ${keypoint4_l_y} 0.0" rpy="0 0 0" />
+      <xacro:pr2_finger_limits_v0/>
+      <dynamics damping="${finger_tip_damping}" />
+      <parent link="${side}_gripper_l_finger_tip_link"/>
+      <child link="${side}_gripper_l_keypoint4_link"/>
+    </joint>
+    <link name="${side}_gripper_l_keypoint4_link"/>
     <joint name="${side}_gripper_l_joint" type="prismatic">
       <parent link="${side}_gripper_l_finger_tip_link"/>
@@ -157,24 +177,4 @@
 	 this link exists twice -->
     <link name="${side}_gripper_l_finger_tip_frame" />
-    <joint name="${side}_gripper_l_keypoint3_joint" type="fixed">
-      <axis xyz="0 0 1" />
-      <!-- <origin xyz="${0.09137} ${-0.00495} 0" rpy="0 0 0" /> -->
-      <origin xyz="${keypoint3_both_x} ${keypoint3_l_y} 0.0" rpy="0 0 0" />
-      <xacro:pr2_finger_limits_v0/>
-      <dynamics damping="${finger_tip_damping}" />
-      <parent link="${side}_gripper_l_finger_tip_frame"/>
-      <child link="${side}_gripper_l_keypoint3_link"/>
-    </joint>
-    <link name="${side}_gripper_l_keypoint3_link"/>
-    <joint name="${side}_gripper_l_keypoint4_joint" type="fixed">
-      <axis xyz="0 0 1" />
-      <!-- <origin xyz="${0.09137} ${-0.00495} 0" rpy="0 0 0" /> -->
-      <origin xyz="${keypoint4_both_x} ${keypoint4_l_y} 0.0" rpy="0 0 0" />
-      <xacro:pr2_finger_limits_v0/>
-      <dynamics damping="${finger_tip_damping}" />
-      <parent link="${side}_gripper_l_finger_tip_frame"/>
-      <child link="${side}_gripper_l_keypoint4_link"/>
-    </joint>
-    <link name="${side}_gripper_l_keypoint4_link"/>
     <!-- Finger tip -->
     <joint name="${prefix}_r_finger_tip_joint" type="revolute">
@@ -209,4 +209,24 @@
       </collision>
     </link>
+        <joint name="${side}_gripper_r_keypoint3_joint" type="fixed">
+      <axis xyz="0 0 1" />
+      <!-- <origin xyz="${0.09137} ${-0.00495} 0" rpy="0 0 0" /> -->
+      <origin xyz="${keypoint3_both_x} ${keypoint3_r_y} 0.0" rpy="0 0 0" />
+      <xacro:pr2_finger_limits_v0/>
+      <dynamics damping="${finger_tip_damping}" />
+      <parent link="${side}_gripper_r_finger_tip_link"/>
+      <child link="${side}_gripper_r_keypoint3_link"/>
+    </joint>
+    <link name="${side}_gripper_r_keypoint3_link"/>
+    <joint name="${side}_gripper_r_keypoint4_joint" type="fixed">
+      <axis xyz="0 0 1" />
+      <!-- <origin xyz="${0.09137} ${-0.00495} 0" rpy="0 0 0" /> -->
+      <origin xyz="${keypoint4_both_x} ${keypoint4_r_y} 0.0" rpy="0 0 0" />
+      <xacro:pr2_finger_limits_v0/>
+      <dynamics damping="${finger_tip_damping}" />
+      <parent link="${side}_gripper_r_finger_tip_link"/>
+      <child link="${side}_gripper_r_keypoint4_link"/>
+    </joint>
+    <link name="${side}_gripper_r_keypoint4_link"/>
     <joint name="${prefix}_r_keypoint1_joint" type="fixed">
       <axis xyz="0 0 1" />
@@ -381,24 +401,4 @@
 	 this link exists twice -->
     <link name="${side}_gripper_r_finger_tip_frame" />
-    <joint name="${side}_gripper_r_keypoint3_joint" type="fixed">
-      <axis xyz="0 0 1" />
-      <!-- <origin xyz="${0.09137} ${-0.00495} 0" rpy="0 0 0" /> -->
-      <origin xyz="${keypoint3_both_x} ${keypoint3_r_y} 0.0" rpy="0 0 0" />
-      <xacro:pr2_finger_limits_v0/>
-      <dynamics damping="${finger_tip_damping}" />
-      <parent link="${side}_gripper_r_finger_tip_frame"/>
-      <child link="${side}_gripper_r_keypoint3_link"/>
-    </joint>
-    <link name="${side}_gripper_r_keypoint3_link"/>
-    <joint name="${side}_gripper_r_keypoint4_joint" type="fixed">
-      <axis xyz="0 0 1" />
-      <!-- <origin xyz="${0.09137} ${-0.00495} 0" rpy="0 0 0" /> -->
-      <origin xyz="${keypoint4_both_x} ${keypoint4_r_y} 0.0" rpy="0 0 0" />
-      <xacro:pr2_finger_limits_v0/>
-      <dynamics damping="${finger_tip_damping}" />
-      <parent link="${side}_gripper_r_finger_tip_frame"/>
-      <child link="${side}_gripper_r_keypoint4_link"/>
-    </joint>
-    <link name="${side}_gripper_r_keypoint4_link"/>
     <!-- extensions -->
     <xacro:pr2_gripper_gazebo_v0 side="${side}" />
